File: hotfire_pcbs/TC-board/TC-board.kicad_sch (KiCad schematic)
At the start: 1 part

Commit message: Progress for TC board.
Parts:
- added J1, J2: JST, symbol Connector:Conn_01x02_Female
- added U1, U2: MAX31856_Breakout, MAX31856_Breakout:MAX31856_Breakout, symbol MAX31856_Breakout:MAX31856_Breakout
- J3: renamed from J?; value Conn_02x18_Row_Letter_First -> PCIE-LP-01-01-F-DV-A-TR; footprint (none) -> SAMTEC_PCIE-LP-01-01-F-DV-A-TR; symbol Connector_Generic:Conn_02x18_Row_Letter_First -> PCIE_Card_Edge:PCIE-LP-01-01-F-DV-A-TR; MANUFACTURER (none) -> Samtec; MAXIMUM_PACKAGE_HEIGHT (none) -> 8.13mm; PARTREV (none) -> B; STANDARD (none) -> Manufacturer Recommendations
Connections:
- net GND: now also J3.A02, J3.A06, J3.A08, J3.A10, J3.A12, J3.A14, J3.A16, J3.A18, J3.B02, J3.B07, J3.B09, J3.B11, J3.B13, J3.B15, U1.9 (GND), U2.9 (GND); no longer J3.a2 (Pin_a2)
- removed net +3.3V: J3.a1 (Pin_a1)
- new net +3V3: J3.B17, J3.B18, U1.11 (VIN), U2.11 (VIN)
- new net SPI_CS_0: J3.B03, U1.5 (CS)
- new net SPI_CS_1: J3.B04, U2.5 (CS)
- new net SPI_MISO: J3.A03, U1.7 (SDO), U2.7 (SDO)
- new net SPI_MOSI: J3.A04, U1.6 (SDI), U2.6 (SDI)
- new net SPI_SCK: J3.B05, U1.8 (SCK), U2.8 (SCK)
- new net TC1_T+: J1.2 (Pin_2), U1.2 (T+)
- new net TC1_T-: J1.1 (Pin_1), U1.1 (T-)
- new net TC2_T+: J2.2 (Pin_2), U2.2 (T+)
- new net TC2_T-: J2.1 (Pin_1), U2.1 (T-)
- no-connect marks 0 -> 21
Other:
- note added: "Thermocouple Amplifier"
- moved on the sheet: J3
