File: le2-daq-new/le2-daq-new.kicad_pcb (KiCad board)
At the start: 2 copper layers, 23 parts, among them J1 RELAY-CONN, J10 PWR-RAIL, J11 PWR-RAIL, J12 PWR-RAIL, J13 PWR-RAIL, J14 PWR-RAIL, J15 PWR-RAIL, J16 PWR-RAIL, J2 PT-CONN, J3 TC-CONN, J4 CAP-CONN, J5 PWR-RAIL, J6 PWR-RAIL, J7 PWR-RAIL, J8 PWR-RAIL, J9 PWR-RAIL, U1 ESP32-DEVKITC-32D

Commit message: owo
Parts:
- added J17: PWR_SUPPLY, Connector_PinHeader_2.54mm:PinHeader_1x02_P2.54mm_Horizontal, F.Cu at (97.1, 125.7)
- J1: footprint Connector_PinHeader_1.00mm:PinHeader_1x10_P1.00mm_Horizontal -> Connector_PinHeader_2.54mm:PinHeader_1x10_P2.54mm_Horizontal
- J10, J11, J12, J13, J14, J15, J16, J5, J6, J7, J8, J9: footprint Connector_PinHeader_1.00mm:PinHeader_1x02_P1.00mm_Horizontal -> Connector_PinHeader_2.54mm:PinHeader_1x02_P2.54mm_Horizontal
- J2: footprint Connector_PinHeader_1.00mm:PinHeader_1x09_P1.00mm_Horizontal -> Connector_PinHeader_2.54mm:PinHeader_1x09_P2.54mm_Horizontal
- J3: footprint Connector_PinHeader_1.00mm:PinHeader_1x06_P1.00mm_Horizontal -> Connector_PinHeader_2.54mm:PinHeader_1x06_P2.54mm_Horizontal
- J4: footprint Connector_PinHeader_1.00mm:PinHeader_1x05_P1.00mm_Horizontal -> Connector_PinHeader_2.54mm:PinHeader_1x05_P2.54mm_Horizontal
- R3: value 100 -> 330
- moved J1 13.9 mm to (158.8, 58.9)
- moved J4 10.3 mm to (93.7, 98.0)
- moved J3 9.86 mm to (93.2, 78.0)
- moved D1 5.89 mm to (114.6, 114.9)
- moved J11 5.89 mm to (148.6, 120.3)
- moved J12 5.89 mm to (116.6, 120.6)
- moved J13 5.89 mm to (158.7, 120.3)
- moved J14 5.89 mm to (127.0, 120.6)
- moved J15 5.89 mm to (137.4, 120.4)
- moved R2 5.89 mm to (108.0, 114.9)
- moved J16 5.89 mm to (106.2, 120.7)
- moved J2 5.21 mm to (102.2, 72.1)
- moved J6 1.79 mm to (112.5, 44.5)
- moved J10 1.79 mm to (156.2, 44.5)
- moved J5 1.79 mm to (103.4, 44.5)
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Routing:
- net +3.3V: track 185.2 -> 219.1 mm
- net 12V: track 64.3 -> 81.0 mm
- net TC2 CS: track 22.2 -> 36.4 mm
- net CS 2: track 20.8 -> 32.2 mm
- net CS 1: track 23.1 -> 34.3 mm
- net CS CLK: track 46.8 -> 57.6 mm
- net TC1 CS: track 21.2 -> 31.8 mm
- net TC CLK: track 50.5 -> 59.1 mm
- net TC SDO: track 22.4 -> 30.9 mm
- net RL 1: track 16.8 -> 11.1 mm
- net RL 2: track 16.1 -> 11.1 mm
- net PT 1: track 18.8 -> 23.2 mm
- net PT 2: track 19.4 -> 23.2 mm
- net PT 3: track 20.1 -> 23.2 mm
- net PT 4: track 20.7 -> 23.2 mm
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Other:
- board outline added: 92.7 x 106 mm
- board text added: "12V"
- board text added: "3.3V"
- board text added: "330"
- board text added: "5K"
- board text added: "GND"
- board text removed: "PWR-RAIL"

Commit message: stash
Parts:
- removed D1, D2: LED, LED_THT:LED_D3.0mm
- removed J10, J11, J12, J13, J14, J15, J16, J6, J7, J8, J9: PWR-RAIL, Connector_PinHeader_2.54mm:PinHeader_1x02_P2.54mm_Horizontal
- removed J17: PWR_SUPPLY, Connector_PinHeader_2.54mm:PinHeader_1x02_P2.54mm_Horizontal
- removed R2: 5K, Resistor_SMD:R_0805_2012Metric_Pad1.20x1.40mm_HandSolder
- removed R3: 330, Resistor_SMD:R_0805_2012Metric_Pad1.20x1.40mm_HandSolder
- added SW1: SW_Push, Jumper:SolderJumper-2_P1.3mm_Bridged2Bar_Pad1.0x1.5mm, F.Cu at (98.8, 131.8)
- J1: footprint Connector_PinHeader_2.54mm:PinHeader_1x10_P2.54mm_Horizontal -> PCIE_1x_Socket:AMPHENOL_10018784-10210TLF
- J2: value PT-CONN -> CAP-CONN; footprint Connector_PinHeader_2.54mm:PinHeader_1x09_P2.54mm_Horizontal -> PCIE_1x_Socket:AMPHENOL_10018784-10210TLF
- J3: footprint Connector_PinHeader_2.54mm:PinHeader_1x06_P2.54mm_Horizontal -> PCIE_1x_Socket:AMPHENOL_10018784-10210TLF
- J4: value CAP-CONN -> HX_CON; footprint Connector_PinHeader_2.54mm:PinHeader_1x05_P2.54mm_Horizontal -> PCIE_1x_Socket:AMPHENOL_10018784-10210TLF
- J5: value PWR-RAIL -> Conn_01x02_Male
- moved J5 106.2 mm to (120.2, 149.4), turned to 180 degrees
- moved R1 73.4 mm to (96.0, 131.8)
- moved J1 67.7 mm to (94.0, 78.5), turned to 90 degrees
- moved G*** 50.8 mm to (136.7, 137.4)
- moved U1 39.7 mm to (116.1, 114.0), turned to 90 degrees
- moved J2 35.4 mm to (135.9, 61.5), turned to 90 degrees
- moved J4 34.9 mm to (122.9, 79.0), turned to 90 degrees
- moved J3 21.7 mm to (110.9, 65.5), turned to -90 degrees
Connections:
- U1 pad 10: TC SDO -> HXLC 1
- U1 pad 11: PT CLK -> HXLC 2
- U1 pad 12: CS 1 -> HX CLK
- U1 pad 15: CS 2 -> unconnected-(U1-Pad15)
- U1 pad 16: unconnected-(U1-Pad16) -> CAP 1
- U1 pad 17: unconnected-(U1-Pad17) -> CAP 2
- U1 pad 2: Net-(R1-Pad1) -> Net-(SW1-Pad2)
- U1 pad 3: PT 1 -> TC CLK
- U1 pad 32: TC CLK -> unconnected-(U1-Pad32)
- U1 pad 35: CS CLK -> CAP CLK
- U1 pad 4: PT 2 -> TC SDO
- U1 pad 5: PT 3 -> TC1 CS
- U1 pad 6: PT 4 -> TC2 CS
- U1 pad 7: PT 5 -> HXPT 1
- U1 pad 8: TC1 CS -> HXPT 2
- U1 pad 9: TC2 CS -> HXPT 3
Routing:
- net +3.3V: track 219.1 -> 0.00 mm
- net 12V: track 81.0 -> 0.00 mm
- net TC CLK: track 59.1 -> 0.00 mm
- net CS CLK: track 57.6 -> 0.00 mm
- net PT CLK: track 44.7 -> 0.00 mm
- net TC2 CS: track 36.4 -> 0.00 mm
- net CS 1: track 34.3 -> 0.00 mm
- net CS 2: track 32.2 -> 0.00 mm
- net TC1 CS: track 31.8 -> 0.00 mm
- net TC SDO: track 30.9 -> 0.00 mm
- net PT 4: track 23.2 -> 0.00 mm
- net PT 2: track 23.2 -> 0.00 mm
- net PT 1: track 23.2 -> 0.00 mm
- net PT 5: track 23.2 -> 0.00 mm
- net PT 3: track 23.2 -> 0.00 mm
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- removed copper zone on B.Cu, net GND
- removed copper zone on F.Cu, net GND
Other:
- board outline removed
- board text removed: "12V"
- board text removed: "12V SUPPLY RAIL"
- board text removed: "3.3V"
- board text removed: "330"
- board text removed: "3V SUPPLY RAIL"
- board text removed: "5K"
- board text removed: "ESP32-DEVKITC-32D"
- board text removed: "GND"
- board text removed: "PT-CONN"
- board text removed: "RELAY-CONN"
- board text removed: "THIS SIDE UP"

Commit message: pcb updates etc
Parts:
- moved J5 13.3 mm to (118.9, 136.1)
- moved G*** 6.37 mm to (130.3, 137.9), turned to 90 degrees
Routing:
- net +3.3V: track 0.00 -> 234.7 mm
- net Net-(SW1-Pad2): track 0.00 -> 4.45 mm
- net Net-(R1-Pad1): track 0.00 -> 2.94 mm
- net CAP 2: track 0.00 -> 1.56 mm
- net GND: vias 25 -> 21
Other:
- board outline added: 62 x 105.9 mm
Changed lines of the file:
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@@
   )
   (footprint "Connector_PinHeader_2.54mm:PinHeader_1x02_P2.54mm_Horizontal" (layer "F.Cu")
-    (at 120.199 149.357 180)
+    (at 118.929 136.149 180)
     (descr "Through hole angled pin header, 1x02, 2.54mm pitch, 6mm pin length, single row")
     (tags "Through hole angled pin header THT 1x02 2.54mm single row")
@@
   )
   (footprint "star:star_8x7" (layer "F.Cu")
-    (at 136.652 137.414)
+    (at 130.302 137.922 90)
     (attr through_hole)
-    (fp_text reference "G***" (at 0 0) (layer "F.SilkS") hide
+    (fp_text reference "G***" (at 0 0 90) (layer "F.SilkS") hide
       (effects (font (size 1.524 1.524) (thickness 0.3)))
     )
-    (fp_text value "LOGO" (at 0.75 0) (layer "F.SilkS") hide
+    (fp_text value "LOGO" (at 0.75 0 90) (layer "F.SilkS") hide
       (effects (font (size 1.524 1.524) (thickness 0.3)))
     )
@@
       (effects (font (size 1 1) (thickness 0.15)))
     )
-    (fp_text user "A1" (at -16.85 -0.65 90) (layer "F.SilkS")
-      (effects (font (size 1 1) (thickness 0.15)))
-    )
-    (fp_text user "B1" (at -16.85 1.75 90) (layer "F.SilkS")
-      (effects (font (size 1 1) (thickness 0.15)))
-    )
-    (fp_text user "A1" (at -16.85 -0.65 90) (layer "F.Fab")
-      (effects (font (size 1 1) (thickness 0.15)))
-    )
-    (fp_text user "B1" (at -16.85 1.75 90) (layer "F.Fab")
-      (effects (font (size 1 1) (thickness 0.15)))
-    )
     (fp_line (start -14.5 -3.7) (end -11.75 -3.7) (layer "F.SilkS") (width 0.127))
     (fp_line (start -14.5 5.1) (end -14.5 -3.7) (layer "F.SilkS") (width 0.127))
@@
       (net 49 "unconnected-(J1-PadB18)") (pinfunction "Pin_b18") (pintype "passive+no_connect"))
   )
-  (gr_rect (start 129.794 132.334) (end 143.51 150.622) (layer "F.SilkS") (width 0.15) (fill none))
-  (gr_text "Ground DAQ\nLE2 Hotfire\n2023" (at 136.398 145.796) (layer "F.SilkS")
+  (gr_rect (start 125.222 144.78) (end 143.51 131.064) (layer "F.SilkS") (width 0.15) (fill none))
+  (gr_rect (start 85.852 46.736) (end 147.828 152.654) (layer "Edge.Cuts") (width 0.1) (fill none))
+  (gr_text "Ground DAQ\nLE2 Hotfire\n2023" (at 138.684 138.176 90) (layer "F.SilkS")
     (effects (font (size 1.27 1.27) (thickness 0.15)))
   )
@@
     (effects (font (size 1 1) (thickness 0.15)))
   )
-  (via (at 132.45 140.576) (size 0.8) (drill 0.4) (layers "F.Cu" "B.Cu") (free) (net 10))
-  (via (at 153.416 166.37) (size 4) (drill 2) (layers "F.Cu" "B.Cu") (free) (net 10))
+  (segment (start 93.472 129.592) (end 93.472 135.128) (width 0.25) (layer "F.Cu") (net 9))
+  (segment (start 117.41 137.668) (end 118.929 136.149) (width 0.25) (layer "F.Cu") (net 9))
+  (segment (start 96.318 126.746) (end 93.472 129.592) (width 0.25) (layer "F.Cu") (net 9))
+  (segment (start 96.318 130.52) (end 96.012 130.826) (width 0.25) (layer "F.Cu") (net 9))
+  (segment (start 96.012 137.668) (end 117.41 137.668) (width 0.25) (layer "F.Cu") (net 9))
+  (segment (start 93.472 135.128) (end 96.012 137.668) (width 0.25) (layer "F.Cu") (net 9))
+  (segment (start 96.318 126.746) (end 96.318 130.52) (width 0.25) (layer "F.Cu") (net 9))
+  (segment (start 99.163 94.131) (end 92.73 100.564) (width 0.25) (layer "B.Cu") (net 9))
+  (segment (start 92.73 97.048) (end 92.73 95.992) (width 0.25) (layer "B.Cu") (net 9))
+  (segment (start 99.314 92.456) (end 92.73 99.04) (width 0.254) (layer "B.Cu") (net 9))
+  (segment (start 96.318 126.746) (end 96.318 125.782) (width 0.25) (layer "B.Cu") (net 9))
+  (segment (start 112.106 53.85) (end 114.419805 53.85) (width 0.25) (layer "B.Cu") (net 9))
+  (segment (start 114.419805 53.85) (end 115.035 54.465195) (width 0.25) (layer "B.Cu") (net 9))
+  (segment (start 96.318 126.746) (end 95.504 126.746) (width 0.25) (layer "B.Cu") (net 9))
+  (segment (start 121.686 90.644) (end 121.686 91.166) (width 0.254) (layer "B.Cu") (net 9))
+  (segment (start 92.73 95.992) (end 92.73 90.136) (width 0.25) (layer "B.Cu") (net 9))
+  (segment (start 134.64 73.118) (end 134.64 92.992) (width 0.25) (layer "B.Cu") (net 9))
+  (segment (start 115.035 54.465195) (end 115.035 74.703) (width 0.25) (layer "B.Cu") (net 9))
+  (segment (start 92.73 98.532) (end 92.73 98.572) (width 0.254) (layer "B.Cu") (net 9))
+  (segment (start 96.318 126.746) (end 92.73 123.158) (width 0.25) (layer "B.Cu") (net 9))
+  (segment (start 121.686 91.166) (end 120.396 92.456) (width 0.254) (layer "B.Cu") (net 9))
+  (segment (start 101.64 88.138) (end 100.985 88.793) (width 0.25) (layer "B.Cu") (net 9))
+  (segment (start 92.73 100.564) (end 92.73 99.294) (width 0.25) (layer "B.Cu") (net 9))
+  (segment (start 134.64 92.992) (end 133.501 94.131) (width 0.25) (layer "B.Cu") (net 9))
+  (segment (start 92.73 123.158) (end 92.73 100.564) (width 0.25) (layer "B.Cu") (net 9))
+  (segment (start 133.501 94.131) (end 99.163 94.131) (width 0.25) (layer "B.Cu") (net 9))
+  (segment (start 100.985 88.753) (end 115.035 74.703) (width 0.25) (layer "B.Cu") (net 9))
+  (segment (start 100.985 88.793) (end 100.985 88.753) (width 0.25) (layer "B.Cu") (net 9))
+  (segment (start 92.73 99.04) (end 92.73 99.294) (width 0.254) (layer "B.Cu") (net 9))
+  (segment (start 92.73 98.572) (end 92.73 97.048) (width 0.25) (layer "B.Cu") (net 9))
+  (segment (start 120.396 92.456) (end 99.314 92.456) (width 0.254) (layer "B.Cu") (net 9))
+  (segment (start 100.985 88.793) (end 92.73 97.048) (width 0.25) (layer "B.Cu") (net 9))
+  (segment (start 92.73 99.294) (end 92.73 98.572) (width 0.25) (layer "B.Cu") (net 9))
+  (via (at 144.78 149.352) (size 4) (drill 2) (layers "F.Cu" "B.Cu") (free) (net 10))
   (via (at 109.59 106.286) (size 0.8) (drill 0.4) (layers "F.Cu" "B.Cu") (free) (net 10))
   (via (at 109.59 103.746) (size 0.8) (drill 0.4) (layers "F.Cu" "B.Cu") (free) (net 10))
-  (via (at 109.59 94.856) (size 0.8) (drill 0.4) (layers "F.Cu" "B.Cu") (free) (net 10))
   (via (at 121.655 95.491) (size 0.8) (drill 0.4) (layers "F.Cu" "B.Cu") (free) (net 10))
-  (via (at 67.31 52.07) (size 4) (drill 2) (layers "F.Cu" "B.Cu") (free) (net 10))
-  (via (at 142.748 131.191) (size 0.8) (drill 0.4) (layers "F.Cu" "B.Cu") (free) (net 10))
-  (via (at 66.04 166.116) (size 4) (drill 2) (layers "F.Cu" "B.Cu") (free) (net 10))
-  (via (at 121.655 91.046) (size 0.8) (drill 0.4) (layers "F.Cu" "B.Cu") (free) (net 10))
+  (via (at 88.646 49.784) (size 4) (drill 2) (layers "F.Cu" "B.Cu") (free) (net 10))
+  (via (at 101.092 140.462) (size 0.8) (drill 0.4) (layers "F.Cu" "B.Cu") (free) (net 10))
+  (via (at 88.646 149.352) (size 4) (drill 2) (layers "F.Cu" "B.Cu") (free) (net 10))
   (via (at 115.305 100.571) (size 0.8) (drill 0.4) (layers "F.Cu" "B.Cu") (free) (net 10))
   (via (at 121.655 103.746) (size 0.8) (drill 0.4) (layers "F.Cu" "B.Cu") (free) (net 10))
-  (via (at 92.456 141.224) (size 0.8) (drill 0.4) (layers "F.Cu" "B.Cu") (free) (net 10))
+  (via (at 92.71 140.716) (size 0.8) (drill 0.4) (layers "F.Cu" "B.Cu") (free) (net 10))
   (via (at 115.305 103.746) (size 0.8) (drill 0.4) (layers "F.Cu" "B.Cu") (free) (net 10))
   (via (at 108.32 140.576) (size 0.8) (drill 0.4) (layers "F.Cu" "B.Cu") (free) (net 10))
   (via (at 115.305 106.286) (size 0.8) (drill 0.4) (layers "F.Cu" "B.Cu") (free) (net 10))
-  (via (at 115.305 94.856) (size 0.8) (drill 0.4) (layers "F.Cu" "B.Cu") (free) (net 10))
   (via (at 121.655 106.286) (size 0.8) (drill 0.4) (layers "F.Cu" "B.Cu") (free) (net 10))
   (via (at 122.29 140.576) (size 0.8) (drill 0.4) (layers "F.Cu" "B.Cu") (free) (net 10))
-  (via (at 153.416 65.278) (size 4) (drill 2) (layers "F.Cu" "B.Cu") (free) (net 10))
+  (via (at 145.034 49.784) (size 4) (drill 2) (layers "F.Cu" "B.Cu") (free) (net 10))
   (via (at 109.59 91.046) (size 0.8) (drill 0.4) (layers "F.Cu" "B.Cu") (free) (net 10))
   (via (at 109.59 100.571) (size 0.8) (drill 0.4) (layers "F.Cu" "B.Cu") (free) (net 10))
@@
   (via (at 115.305 140.576) (size 0.8) (drill 0.4) (layers "F.Cu" "B.Cu") (free) (net 10))
   (via (at 115.305 91.046) (size 0.8) (drill 0.4) (layers "F.Cu" "B.Cu") (free) (net 10))
+  (segment (start 96.362 132.476) (end 98.806 132.476) (width 0.25) (layer "F.Cu") (net 24))
+  (segment (start 96.012 132.826) (end 96.362 132.476) (width 0.25) (layer "F.Cu") (net 24))
+  (segment (start 138.063 125.641) (end 136.958 126.746) (width 0.25) (layer "F.Cu") (net 68))
+  (segment (start 124.186 86.644) (end 124.257 86.715) (width 0.25) (layer "F.Cu") (net 135))
+  (segment (start 98.858 131.124) (end 98.806 131.176) (width 0.25) (layer "F.Cu") (net 150))
+  (segment (start 98.858 126.746) (end 98.858 131.124) (width 0.25) (layer "F.Cu") (net 150))
 )

Commit message: CORE PCB DONE
Parts:
- added J6: TEST-POINT, Connector_PinHeader_2.54mm:PinHeader_1x19_P2.54mm_Horizontal, F.Cu at (140.7, 78.2)
- added J7: TEST-POINT, Connector_PinHeader_2.54mm:PinHeader_1x19_P2.54mm_Horizontal, F.Cu at (92.3, 123.9)
- J1: value RELAY-CONN -> PCIE_CONN; footprint PCIE_1x_Socket:AMPHENOL_10018784-10210TLF -> PCIE-LP-01-01-F-DV-A-TR:SAMTEC_PCIE-LP-01-01-F-DV-A-TR
- J2: value CAP-CONN -> PCIE_CONN; footprint PCIE_1x_Socket:AMPHENOL_10018784-10210TLF -> PCIE-LP-01-01-F-DV-A-TR:SAMTEC_PCIE-LP-01-01-F-DV-A-TR
- J3: value TC-CONN -> PCIE_CONN; footprint PCIE_1x_Socket:AMPHENOL_10018784-10210TLF -> PCIE-LP-01-01-F-DV-A-TR:SAMTEC_PCIE-LP-01-01-F-DV-A-TR
- J4: value HX_CON -> PCIE_CONN; footprint PCIE_1x_Socket:AMPHENOL_10018784-10210TLF -> PCIE-LP-01-01-F-DV-A-TR:SAMTEC_PCIE-LP-01-01-F-DV-A-TR
- SW1: value SW_Push -> EN_HIGH
- moved J2 86.4 mm to (189.7, 129.1), turned to 0 degrees
- moved J3 82.4 mm to (189.2, 91.1), turned to 0 degrees
- moved J1 82.4 mm to (176.2, 74.2), turned to 0 degrees
- moved J5 74.0 mm to (72.9, 78.2), turned to -90 degrees
- moved G*** 64.7 mm to (70.4, 113.5), turned to 0 degrees
- moved J4 59.7 mm to (174.2, 109.5), turned to 0 degrees
- moved R1 53.9 mm to (99.3, 78.0), turned to 0 degrees
- moved SW1 51.1 mm to (99.3, 80.8), turned to 0 degrees
- moved U1 16.0 mm to (117.1, 98.0), turned to 0 degrees
Connections:
- net Net-(SW1-Pad2) renamed EN
- J1 pad A10: unconnected-(J1-PadA10) -> GND
- J1 pad A11: unconnected-(J1-PadA11) -> HX CLK
- J1 pad A12: unconnected-(J1-PadA12) -> CAP 2
- J1 pad A13: unconnected-(J1-PadA13) -> PHOTORES
- J1 pad A14: unconnected-(J1-PadA14) -> GND
- J1 pad A15: unconnected-(J1-PadA15) -> GND
- J1 pad A16: unconnected-(J1-PadA16) -> EXTRA
- J1 pad A17: unconnected-(J1-PadA17) -> +5V
- J1 pad A18: unconnected-(J1-PadA18) -> +5V
- J1 pad B10: unconnected-(J1-PadB10) -> HX 6
- J1 pad B11: unconnected-(J1-PadB11) -> HX 8
- J1 pad B12: unconnected-(J1-PadB12) -> GND
- J1 pad B13: unconnected-(J1-PadB13) -> CAP 1
- J1 pad B14: unconnected-(J1-PadB14) -> RL INT
- J1 pad B15: unconnected-(J1-PadB15) -> CAP CLK
- J1 pad B16: unconnected-(J1-PadB16) -> GND
- J1 pad B17: unconnected-(J1-PadB17) -> +3.3V
- J1 pad B18: unconnected-(J1-PadB18) -> +3.3V
- J2 pad A10: unconnected-(J2-PadA10) -> GND
- J2 pad A11: unconnected-(J2-PadA11) -> HX CLK
- J2 pad A12: unconnected-(J2-PadA12) -> CAP 2
- J2 pad A13: unconnected-(J2-PadA13) -> PHOTORES
- J2 pad A14: unconnected-(J2-PadA14) -> GND
- J2 pad A15: unconnected-(J2-PadA15) -> GND
- J2 pad A16: unconnected-(J2-PadA16) -> EXTRA
- J2 pad A17: unconnected-(J2-PadA17) -> +5V
- J2 pad A18: unconnected-(J2-PadA18) -> +5V
- J2 pad B10: unconnected-(J2-PadB10) -> HX 6
- J2 pad B11: unconnected-(J2-PadB11) -> HX 8
- J2 pad B12: unconnected-(J2-PadB12) -> GND
- J2 pad B13: unconnected-(J2-PadB13) -> CAP 1
- J2 pad B14: unconnected-(J2-PadB14) -> RL INT
- J2 pad B15: unconnected-(J2-PadB15) -> CAP CLK
- J2 pad B16: unconnected-(J2-PadB16) -> GND
- J2 pad B17: unconnected-(J2-PadB17) -> +3.3V
- J2 pad B18: unconnected-(J2-PadB18) -> +3.3V
- J3 pad A10: unconnected-(J3-PadA10) -> GND
- J3 pad A11: unconnected-(J3-PadA11) -> HX CLK
- J3 pad A12: unconnected-(J3-PadA12) -> CAP 2
- J3 pad A13: unconnected-(J3-PadA13) -> PHOTORES
- J3 pad A14: unconnected-(J3-PadA14) -> GND
- J3 pad A15: unconnected-(J3-PadA15) -> GND
- J3 pad A16: unconnected-(J3-PadA16) -> EXTRA
- J3 pad A17: unconnected-(J3-PadA17) -> +5V
- J3 pad A18: unconnected-(J3-PadA18) -> +5V
- J3 pad B10: unconnected-(J3-PadB10) -> HX 6
- J3 pad B11: unconnected-(J3-PadB11) -> HX 8
- J3 pad B12: unconnected-(J3-PadB12) -> GND
- J3 pad B13: unconnected-(J3-PadB13) -> CAP 1
- J3 pad B14: unconnected-(J3-PadB14) -> RL INT
- J3 pad B15: unconnected-(J3-PadB15) -> CAP CLK
- J3 pad B16: unconnected-(J3-PadB16) -> GND
- J3 pad B17: unconnected-(J3-PadB17) -> +3.3V
- J3 pad B18: unconnected-(J3-PadB18) -> +3.3V
- J4 pad A10: unconnected-(J4-PadA10) -> GND
- J4 pad A11: unconnected-(J4-PadA11) -> HX CLK
- J4 pad A12: unconnected-(J4-PadA12) -> CAP 2
- J4 pad A13: unconnected-(J4-PadA13) -> PHOTORES
- J4 pad A14: unconnected-(J4-PadA14) -> GND
- J4 pad A15: unconnected-(J4-PadA15) -> GND
- J4 pad A16: unconnected-(J4-PadA16) -> EXTRA
- J4 pad A17: unconnected-(J4-PadA17) -> +5V
- J4 pad A18: unconnected-(J4-PadA18) -> +5V
- J4 pad B10: unconnected-(J4-PadB10) -> HX 6
- J4 pad B11: unconnected-(J4-PadB11) -> HX 8
- J4 pad B12: unconnected-(J4-PadB12) -> GND
- J4 pad B13: unconnected-(J4-PadB13) -> CAP 1
- J4 pad B14: unconnected-(J4-PadB14) -> RL INT
- J4 pad B15: unconnected-(J4-PadB15) -> CAP CLK
- J4 pad B16: unconnected-(J4-PadB16) -> GND
- J4 pad B17: unconnected-(J4-PadB17) -> +3.3V
- J4 pad B18: unconnected-(J4-PadB18) -> +3.3V
- U1 pad 10: HXLC 1 -> HX 8
- U1 pad 11: HXLC 2 -> HX CLK
- U1 pad 12: HX CLK -> EXTRA
- U1 pad 19: unconnected-(U1-Pad19) -> +5V
- U1 pad 21: RL 1 -> RL INT
- U1 pad 22: RL 2 -> RL SCL
- U1 pad 25: RL 3 -> RL SDA
- U1 pad 27: RL 4 -> PHOTORES
- U1 pad 28: RL 5 -> TC2 CS
- U1 pad 29: RL 6 -> TC1 CS
- U1 pad 3: TC CLK -> HX 1
- U1 pad 30: RL 7 -> TC SDO
- U1 pad 31: RL 8 -> TC CLK
- U1 pad 35: CAP CLK -> unconnected-(U1-Pad35)
- U1 pad 38: unconnected-(U1-Pad38) -> CAP CLK
- U1 pad 4: TC SDO -> HX 2
- U1 pad 5: TC1 CS -> HX 3
- U1 pad 6: TC2 CS -> HX 4
- U1 pad 7: HXPT 1 -> HX 5
- U1 pad 8: HXPT 2 -> HX 6
- U1 pad 9: HXPT 3 -> HX 7
Routing:
- net HX CLK: track 0.00 -> 318.1 mm, vias 0 -> 3
- net HX 6: track 0.00 -> 280.2 mm, vias 0 -> 6
- net EXTRA: track 0.00 -> 194.8 mm, vias 0 -> 4
- net PHOTORES: track 0.00 -> 192.8 mm, vias 0 -> 6
- net HX 8: track 0.00 -> 187.6 mm, vias 0 -> 7
- net CAP 1: track 0.00 -> 182.5 mm, vias 0 -> 8
- net +5V: track 0.00 -> 166.5 mm, vias 0 -> 4
- net CAP 2: track 1.56 -> 165.1 mm, vias 0 -> 7
- net RL INT: track 0.00 -> 131.3 mm, vias 0 -> 6
- net CAP CLK: track 0.00 -> 128.4 mm, vias 0 -> 6
- net +3.3V: track 234.7 -> 181.6 mm, vias 0 -> 6
- net HX 7: track 0.00 -> 12.2 mm
- net HX 5: track 0.00 -> 12.2 mm
- net HX 4: track 0.00 -> 12.2 mm
- net HX 3: track 0.00 -> 12.2 mm
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- added copper zone on B.Cu, net (none)
- added copper zone on F.Cu, net GND
Other:
- board size 62 x 105.9 mm -> 161.3 x 88.4 mm
- board text removed: "CAP-CONN"
- board text removed: "TC-CONN"
