File: hotfire_pcbs/relay-board/relay-board.kicad_sch (KiCad schematic)
At the start: 5 parts, among them J1 Conn_02x18_Row_Letter_First, U1 Relay_Board, U2 Relay_Board, U3 Relay_Board, U4 Relay_Board

Commit message: relay schematic
Parts:
- added R1, R10, R11, R12, R15, R16, R17, R18, R19, R2, R20, R23, R24, R25, R26, R27, R28, R3, R31, R32, R4, R7, R8, R9: 1k, symbol Device:R_Small
- added R13, R14, R21, R22, R29, R30, R5, R6: 2k, symbol Device:R_Small
- added U10, U11, U12, U13, U5, U6, U8, U9: LM741, symbol Amplifier_Operational:LM741
- added U7: PCF8575_Breakout, symbol PCF87575:PCF8575_Breakout
- J1: value Conn_02x18_Row_Letter_First -> PCIE_CONN; footprint (none) -> PCIE-LP-01-01-F-DV-A-TR:SAMTEC_PCIE-LP-01-01-F-DV-A-TR
Connections:
- net +3.3V: now also J1.B17 (Pin_b17), J1.B18 (Pin_b18), U7.12 (VCC), U7.17 (VDD), U7.9 (VDD); no longer J1.a1 (Pin_a1), U1.1 (VCC), U2.1 (VCC), U3.1 (VCC), U4.1 (VCC)
- net GND: now also J1.A10 (Pin_a10), J1.A14 (Pin_a14), J1.A15 (Pin_a15), J1.A2 (Pin_a2), J1.A4 (Pin_a4), J1.A7 (Pin_a7), J1.B12 (Pin_b12), J1.B16 (Pin_b16), J1.B2 (Pin_b2), J1.B6 (Pin_b6), J1.B9 (Pin_b9), R10.1, R12.1, R15.2, R16.2, R18.1, R2.1, R20.1, R23.2, R24.2, R26.1, R28.1, R31.2, R32.2, R4.1, R7.2, R8.2, U10.4 (V-), U11.4 (V-), U12.4 (V-), U13.4 (V-), U5.4 (V-), U6.4 (V-), U7.10 (GND), U7.11 (GND), U7.16 (GND), U8.4 (V-), U9.4 (V-); no longer J1.a2 (Pin_a2)
- net REL 1: now also R5.2, R7.1, U5.6
- net REL 2: now also R6.2, R8.1, U6.6
- net REL 3: now also R13.2, R15.1, U8.6
- net REL 4: now also R14.2, R16.1, U9.6
- net REL 5: now also R21.2, R23.1, U10.6
- net REL 6: now also R22.2, R24.1, U11.6
- net REL 7: now also R29.2, R31.1, U12.6
- net REL 8: now also R30.2, R32.1, U13.6
- new net: R28.2, R30.1, U13.2 (-)
- new net: R12.2, R14.1, U9.2 (-)
- new net: R18.2, R21.1, U10.2 (-)
- new net: R2.2, R5.1, U5.2 (-)
- new net: R26.2, R29.1, U12.2 (-)
- new net: R4.2, R6.1, U6.2 (-)
- new net: R20.2, R22.1, U11.2 (-)
- new net: R10.2, R13.1, U8.2 (-)
- new net +5V: J1.A17 (Pin_a17), J1.A18 (Pin_a18), R1.1, R11.1, R17.1, R19.1, R25.1, R27.1, R3.1, R9.1, U1.1 (VCC), U10.7 (V+), U11.7 (V+), U12.7 (V+), U13.7 (V+), U2.1 (VCC), U3.1 (VCC), U4.1 (VCC), U5.7 (V+), U6.7 (V+), U8.7 (V+), U9.7 (V+)
- new net P0: R1.2, U5.3 (+), U7.18 (P00)
- new net P1: R3.2, U6.3 (+), U7.19 (P01)
- new net P2: R9.2, U7.20 (P02), U8.3 (+)
- new net P3: R11.2, U7.21 (P03), U9.3 (+)
- new net P4: R17.2, U10.3 (+), U7.22 (P04)
- new net P5: R19.2, U11.3 (+), U7.23 (P05)
- new net P6: R25.2, U12.3 (+), U7.24 (P06)
- new net P7: R27.2, U13.3 (+), U7.25 (P07)
- new net RL INT: J1.B14 (Pin_b14), U7.15 (INT)
- new net RL SCL: J1.B1 (Pin_b1), U7.14 (SCL)
- new net RL SDA: J1.A1 (Pin_a1), U7.13 (SDA)
- no-connect marks 0 -> 42
Other:
- moved on the sheet: U1, U2, U3, U4
